File: Hardware/LaserScanner.sch (EAGLE design)
At the start: 35 parts, among them J1 USB, Q1 MBT3904DW1T1, U1 ESP-WROOM-32, U2 3.3V, U3 CH340C

Commit message: Added DAC circuits and power interlocks
Parts:
- added D6, D7: 3A/10V/280mV, SparkFun-DiscreteSemi:DIODE-SCHOTTKY-BAT60A
- added J2: SHTDWN, SparkFun-Connectors:CONN_021X02_NO_SILK
- added J3: KEYSWITCH, SparkFun-Connectors:CONN_021X02_NO_SILK
- added J4: (no value), SparkFun-Connectors:CONN_01PTH_NO_SILK_YES_STOP
- added J5: ESTOP, SparkFun-Connectors:CONN_021X02_NO_SILK
- added JP1: JUMPER-SMT_2_NC_TRACE_SILK, SparkFun-Jumpers:JUMPER-SMT_2_NC_TRACE_SILK
- added R11, R12, R13, R14, R15, R16, R17, R18, R19, R20, R21, R22: 10k, SparkFun-Resistors:10KOHM-0603-1/10W-1%
- R6: value 510 -> 3.3k; device SparkFun-Resistors:510OHM-2010-1/2W-5% -> SparkFun-Resistors:3.3KOHM-0603-1/10W-1%
Connections:
- new net AGND: JP1.1, U$1.AGND, U$2.AGND
- new net AUX_OUT: J4.1, R14.2, U$3.VOUTD
- new net GX_!CS: R17.1, U$2.!CS
- new net GX_!LDAC: R18.1, U$2.!LDAC
- new net GX_!RST: U$2.!RST
- new net GX_OUT: U$2.VOUT
- new net GY_!CS: R19.1, U$1.!CS
- new net GY_!LDAC: R20.1, U$1.!LDAC
- new net GY_!RST: U$1.!RST
- new net GY_OUT: U$1.VOUT
- new net G_MOSI: U$1.SDI, U$2.SDI
- new net G_SCLK: U$1.SCLK, U$2.SCLK
- new net LASER_B: R13.2, U$3.VOUTC
- new net LASER_G: R12.2, U$3.VOUTB
- new net LASER_R: R11.2, U$3.VOUTA
- new net L_!CLR: R15.1, U$3.!CLR
- new net L_!LDAC: R21.1, U$3.!LDAC
- new net L_!SYNC: R22.1, U$3.!SYNC
- new net L_MOSI: U$3.SDIN
- new net L_SCLK: U$3.SCLK
- new net N$7: C4.1, D6.A, U$5.VOUT
- new net N$9: J3.2, J5.1
- new net VCC: J2.1, J5.2
- new net VCC_SWITCHED: C5.1, J3.1, U$4.VIN+
- new net VREFH: U$1.VREFH-F, U$1.VREFH-S, U$2.VREFH-F, U$2.VREFH-S
- new net VREFL: U$1.VREFL-F, U$1.VREFL-S, U$2.VREFL-F, U$2.VREFL-S
- net -12V: now also U$1.VSS, U$2.VSS
- net 12V: now also U$1.VCC, U$2.VCC
- net 3.3V: now also R15.2, R17.2, R18.2, R19.2, R20.2, R21.2, R22.2, U$1.RSTSEL, U$1.VDD, U$2.RSTSEL, U$2.VDD
- net 5V: now also C8.1, D6.C, D7.C, U$3.REFIN, U$3.VDD, U2.EN, U2.IN; no longer C4.1, U$5.VOUT
- net GND: now also JP1.2, R11.1, R12.1, R13.1, R14.1, R16.1, U$1.DGND, U$2.DGND, U$3.GND, U$3.POR
- net N$2: now also R16.2, U$3.SDO; no longer C5.1, U$4.VIN+
- net N$4: now also R6.2; no longer R6.1
- net SHTDWN: now also J2.2, R6.1; no longer R6.2
- net V_USB: now also D7.A; no longer C8.1, U2.EN, U2.IN
Other:
- note added: "3.3V control signal - 1 volt transistor drop and 0.3 volts diode drop is 2V, and required current is 6mA so we choose a 330 ohm resistor JK. If the micro has to supply 3.3V to keep the regulator on then when it turns off the micro will die and the regulator will turn back on causing an oscillation of on and off that would be BAD So then let's just expose a pair of nets that can be connected exter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"
- note added: "?"
- note added: "Here's a *reminder* that somewhere along the line AGND and GND need to be connected. But how to reduce noise from GND on AGND... some kind of filter?"
- note added: "Pull down resistors on laser level channels is an attempt to fail-safe the laser output"
- note added: "Safety feature brainstorm: - Keyed power switch - Emergency stop switch external stop signal (to allow for galvo movement detector later)"
- moved on the sheet: C1, C4, C8, C9, D1, D4, D5, R10, R2, R6, U$1, U$3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

Commit message: Add KILL signal and VREF delay
Parts:
- added C10, C11: 10uF, SparkFun-Capacitors:10UF-1210-50V-20%
- added J6, J7: (no value), SparkFun-Connectors:CONN_06NO_SILK_FEMALE_PTH
- added JP2, JP3: JUMPER-SMT_2_NO_SILK, SparkFun-Jumpers:JUMPER-SMT_2_NO_SILK
- added Q4: 2.5A/30V/105mΩ, SparkFun-DiscreteSemi:MOSFET_PCH-DMG2307L
- added R23, R24, R25, R26, R27: 10k, SparkFun-Resistors:10KOHM-0603-1/10W-1%
- J2: value SHTDWN -> !KILL!
- J4: device SparkFun-Connectors:CONN_01PTH_NO_SILK_YES_STOP -> SparkFun-Connectors:CONN_06NO_SILK_FEMALE_PTH
Connections:
- removed net MISO: U1.MISO_H/IO12
- removed net MOSI: U1.MOSI_H/IO13
- removed net SCLK: U1.SCK_H/IO14
- new net !KILL: J2.2, Q4.G, R27.2
- new net N$11: U1.CS0_V/IO5
- new net N$22: U1.XTAL_P/IO32
- new net N$23: U1.XTAL_N/IO33
- new net N$24: U1.IO34
- new net N$25: U1.IO35
- new net N$8: U1.IO4
- net -12V: now also JP3.1, R23.1
- net 12V: now also JP2.1, R24.1
- net 3.3V: now also R25.2, R26.2
- net AGND: now also C10.2, C11.2, J7.1, J7.2, J7.3, J7.4, J7.5, J7.6
- net AUX_OUT: now also J6.6; no longer J4.1
- net GND: now also J4.1, J4.2, J4.3, J4.4, J4.5, J4.6, R27.1
- net GX_!CS: now also U1.IO21
- net GX_!LDAC: now also U1.MISO_V/IO19
- net GX_!RST: now also R25.1, U1.IO22
- net GX_OUT: now also J6.1
- net GY_!CS: now also U1.IO16
- net GY_!LDAC: now also U1.CS0_H/IO15
- net GY_!RST: now also R26.1, U1.IO17
- net GY_OUT: now also J6.2
- net G_MOSI: now also U1.MOSI_H/IO13
- net G_SCLK: now also U1.SCK_H/IO14
- net LASER_B: now also J6.5
- net LASER_G: now also J6.4
- net LASER_R: now also J6.3
- net L_!CLR: now also U1.IO25
- net L_!LDAC: now also U1.IO27
- net L_!SYNC: now also U1.IO26
- net L_MOSI: now also U1.MOSI_V/IO23
- net L_SCLK: now also U1.SCK_V/IO18
- net SHTDWN: now also Q4.D; no longer J2.2
- net VCC: now also Q4.S
- net VREFH: now also C10.1, JP2.2, R24.2
- net VREFL: now also C11.1, JP3.2, R23.2
Other:
- note added: "!KILL! is an externally manipulatable signal that is used to immediately shut-down, failsafe, and de-energize (or whatever terminology you prefer) the system. GND and VCC are provided for reference. Pull-down prefers the safe(r) state"
- note added: "This makes SHTDWN high when !KILL! is low (active) AND it uses the always on VCC voltage (so it can keep everything turned off"
- note added: "This pair of low pass filters are intended to make the VREF sources come up more slowly than the +/-12V nets. This is by request of the datasheet for the DAC8871's Note: values are as of yet uncalculated!"
- note added: "ToDo: - DAC control circuits - Interlocks and safety - Power in connectors - DAC out connectors - Additional interfaces? 1/3/19 - keep considering more safety features - make a table of VIN requirements - try to make the low pass filters a reasonable time constant"
- note removed: "ToDo: - DAC control circuits - Interlocks and safety - Power in connectors - DAC out connectors - Additional interfaces?"
- moved on the sheet: J2

Commit message: RC calculations
Parts:
- removed JP1: JUMPER-SMT_2_NC_TRACE_SILK, SparkFun-Jumpers:JUMPER-SMT_2_NC_TRACE_SILK
- added C12, C13, C14, C15, C16, C17: 1.0uF, SparkFun-Capacitors:1.0UF-0603-16V-10%-X7R
- added C18, C19, C20, C21, C22: 10uF, SparkFun-Capacitors:10UF-POLAR-EIA3216-16V-10%(TANT)
- added D8: GREEN, SparkFun-LED:LED-GREEN0603
- added D9: Yellow, SparkFun-LED:LED-YELLOW0603
- added J8: Power Input, SparkFun-Connectors:CONN_021X02_NO_SILK
- added R28, R29: 1k, SparkFun-Resistors:1KOHM-0603-1/10W-1%
- added R30, R31: 10k, SparkFun-Resistors:10KOHM-0603-1/10W-1%
Connections:
- new net N$13: D8.A, R28.1
- new net N$14: D9.A, R29.1
- new net N$15: R24.2, R30.1
- new net N$16: R23.2, R31.1
- net -12V: now also C19.+, C21.+
- net 12V: now also C18.+, C20.+
- net 3.3V: now also C17.1, R28.2, R29.2
- net 5V: now also C16.1, C22.+
- net AGND: now also C12.2, C13.2, C14.2, C15.2; no longer C10.2, C11.2, J7.1, J7.2, J7.3, J7.4, J7.5, J7.6, JP1.1, U$1.AGND, U$2.AGND
- net GND: now also C10.2, C11.2, C16.2, C17.2, C18.-, C19.-, C20.-, C21.-, C22.-, J7.1, J7.2, J7.3, J7.4, J7.5, J7.6, J8.2, U$1.AGND, U$2.AGND; no longer JP1.2
- net RXI: now also D9.C
- net TXO: now also D8.C
- net VCC: now also J8.1
- net VREFH: now also C13.1, C15.1, R30.2; no longer R24.2
- net VREFL: now also C12.1, C14.1, R31.2; no longer R23.2
Other:
- note added: "This pair of low pass filters are intended to make the VREF sources come up more slowly than the +/-12V nets. This is by request of the datasheet for the DAC8871's Note: values are as of yet uncalculated! Now I've calculated that with r*c = 0.2 we will reach 90% desired voltage in 0.45 seconds and after 1 second the voltage will be 99.6% of full"
- note removed: "Here's a *reminder* that somewhere along the line AGND and GND need to be connected. But how to reduce noise from GND on AGND... some kind of filter?"
- note removed: "This pair of low pass filters are intended to make the VREF sources come up more slowly than the +/-12V nets. This is by request of the datasheet for the DAC8871's Note: values are as of yet uncalculated!"
- moved on the sheet: C10, C11

Commit message: Push to work from laptop
Parts:
- removed C11, C5: 10uF, SparkFun-Capacitors:10UF-1210-50V-20%
- added R32: 10k, SparkFun-Resistors:10KOHM-0603-1/10W-1%
- added S1: RESET, SparkFun-Switches:MOMENTARY-SWITCH-SPST-2-SMD-4.6X2.8MM
- added S2: 0, SparkFun-Switches:MOMENTARY-SWITCH-SPST-2-SMD-4.6X2.8MM
- C1, C10, C4: device SparkFun-Capacitors:10UF-1210-50V-20% -> SparkFun-Capacitors:10UF-POLAR-EIA3216-16V-10%(TANT)
- U$5: value R-78E3.3-1.0 -> 12to5
Connections:
- removed net AGND: C12.2, C13.2, C14.2, C15.2
- net -12V: no longer C21.+
- net 0: now also R32.1, S2.3, S2.4
- net 12V: now also C1.+; no longer C1.1, C20.+
- net 3.3V: now also R32.2
- net GND: now also C1.-, C10.-, C12.2, C13.2, C14.2, C15.2, C21.+, C4.-, S1.1, S1.2, S2.1, S2.2; no longer C1.2, C10.2, C11.2, C21.-, C4.2, C5.2
- net N$7: now also C4.+; no longer C4.1
- net RESET: now also S1.3, S1.4
- net VCC_SWITCHED: now also C10.+; no longer C5.1
- net VREFH: now also C20.+; no longer C10.1
- net VREFL: now also C21.-; no longer C11.1
Other:
- moved on the sheet: C18, C19, C20, C21, D2, D3, D7, R1, R3, R4, R5

Commit message: Made a significant push on routing the board
Parts:
- removed R32: 10k, SparkFun-Resistors:10KOHM-0603-1/10W-1%
- removed S1: RESET, SparkFun-Switches:MOMENTARY-SWITCH-SPST-2-SMD-4.6X2.8MM
- removed S2: 0, SparkFun-Switches:MOMENTARY-SWITCH-SPST-2-SMD-4.6X2.8MM
- added R33: 10k, SparkFun-Resistors:10KOHM-0603-1/10W-1%
- added S3: USW2, SparkFun-Switches:MOMENTARY-SWITCH-SPST-SMD-5.2-REDUNDANT
- added S4: USW3, SparkFun-Switches:MOMENTARY-SWITCH-SPST-SMD-5.2-REDUNDANT
Connections:
- net -12V: now also C19.-; no longer C19.+
- net 0: now also R33.1, S3.1; no longer R32.1, S2.3, S2.4
- net 3.3V: now also R33.2; no longer R32.2
- net GND: now also C19.+, S3.2, S4.2; no longer C19.-, S1.1, S1.2, S2.1, S2.2
- net LASER_B: now also J6.3; no longer J6.5
- net LASER_G: now also J6.5; no longer J6.4
- net LASER_R: now also J6.4; no longer J6.3
- net RESET: now also S4.1; no longer S1.3, S1.4
Other:
- moved on the sheet: C19

Commit message: Added silk, optimized ground planes, and cammed
Parts:
- removed J4: (no value), SparkFun-Connectors:CONN_06NO_SILK_FEMALE_PTH
- added D10, D11: BLUE, SparkFun-LED:LED-BLUE0603
- added R32, R34: 1k, SparkFun-Resistors:1KOHM-0603-1/10W-1%
- added R35: 100, SparkFun-Resistors:100OHM-0603-1/4W-5%
Connections:
- removed net N$24: U1.IO34
- removed net N$25: U1.IO35
- new net N$17: D10.C, R32.2
- new net N$18: D11.C, R34.2
- new net ULED1: D10.A, U1.IO34
- new net ULED2: D11.A, U1.IO35
- net GND: now also R32.1, R34.1, R35.1; no longer J4.1, J4.2, J4.3, J4.4, J4.5, J4.6
- net N$7: now also R35.2
Other:
- moved on the sheet: D1, R2, S4

Commit message: stop using input only pins for led outputs
Connections:
- removed net N$11: U1.CS0_V/IO5
- removed net N$22: U1.XTAL_P/IO32
- removed net N$23: U1.XTAL_N/IO33
- removed net N$8: U1.IO4
- net ULED1: now also U1.XTAL_P/IO32; no longer U1.IO34
- net ULED2: now also U1.XTAL_N/IO33; no longer U1.IO35
Changed lines of the file:
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@@
 <?xml version="1.0" encoding="utf-8"?>
 <!DOCTYPE eagle SYSTEM "eagle.dtd">
-<eagle version="9.1.3">
+<eagle version="9.2.0">
 <drawing>
 <settings>
-<setting alwaysvectorfont="yes"/>
+<setting alwaysvectorfont="no"/>
 <setting verticaltext="up"/>
 </settings>
@@
 <attribute name="VALUE" x="53.34" y="139.446" size="1.778" layer="96" rot="MR0" align="top-center"/>
 </instance>
-<instance part="D10" gate="G$1" x="30.48" y="160.02"/>
-<instance part="D11" gate="G$1" x="43.18" y="160.02"/>
+<instance part="D10" gate="G$1" x="30.48" y="160.02">
+<attribute name="NAME" x="27.051" y="155.448" size="1.778" layer="95" font="vector" rot="R90"/>
+<attribute name="VALUE" x="32.385" y="155.448" size="1.778" layer="96" font="vector" rot="R90" align="top-left"/>
+</instance>
+<instance part="D11" gate="G$1" x="43.18" y="160.02">
+<attribute name="NAME" x="39.751" y="155.448" size="1.778" layer="95" font="vector" rot="R90"/>
+<attribute name="VALUE" x="45.085" y="155.448" size="1.778" layer="96" font="vector" rot="R90" align="top-left"/>
+</instance>
 <instance part="R32" gate="G$1" x="30.48" y="147.32" rot="R90">
 <attribute name="NAME" x="28.956" y="147.32" size="1.778" layer="95" font="vector" rot="R90" align="bottom-center"/>
@@
 <attribute name="VALUE" x="43.18" y="136.906" size="1.778" layer="96" rot="MR0" align="top-center"/>
 </instance>
-<instance part="R35" gate="G$1" x="162.56" y="76.2" rot="R90"/>
+<instance part="R35" gate="G$1" x="162.56" y="76.2" rot="R90">
+<attribute name="NAME" x="161.036" y="76.2" size="1.778" layer="95" font="vector" rot="R90" align="bottom-center"/>
+<attribute name="VALUE" x="164.084" y="76.2" size="1.778" layer="96" font="vector" rot="R90" align="top-center"/>
+</instance>
 <instance part="GND27" gate="1" x="162.56" y="66.04">
 <attribute name="VALUE" x="162.56" y="65.786" size="1.778" layer="96" align="top-center"/>
@@
 </segment>
 </net>
-<net name="N$8" class="0">
-<segment>
-<pinref part="U1" gate="G$1" pin="IO4"/>
-<wire x1="63.5" y1="241.3" x2="60.96" y2="241.3" width="0.1524" layer="91"/>
-</segment>
-</net>
-<net name="N$11" class="0">
-<segment>
-<pinref part="U1" gate="G$1" pin="CS0_V/IO5"/>
-<wire x1="63.5" y1="238.76" x2="60.96" y2="238.76" width="0.1524" layer="91"/>
-</segment>
-</net>
-<net name="N$22" class="0">
-<segment>
-<pinref part="U1" gate="G$1" pin="XTAL_P/IO32"/>
-<wire x1="63.5" y1="198.12" x2="60.96" y2="198.12" width="0.1524" layer="91"/>
-</segment>
-</net>
-<net name="N$23" class="0">
-<segment>
-<pinref part="U1" gate="G$1" pin="XTAL_N/IO33"/>
-<wire x1="63.5" y1="195.58" x2="60.96" y2="195.58" width="0.1524" layer="91"/>
-</segment>
-</net>
 <net name="!KILL" class="0">
 <segment>
@@
 </segment>
 <segment>
-<pinref part="U1" gate="G$1" pin="IO34"/>
-<wire x1="63.5" y1="193.04" x2="60.96" y2="193.04" width="0.1524" layer="91"/>
-<label x="63.5" y="193.04" size="1.27" layer="95" xref="yes"/>
+<wire x1="63.5" y1="198.12" x2="60.96" y2="198.12" width="0.1524" layer="91"/>
+<label x="63.5" y="198.12" size="1.27" layer="95" xref="yes"/>
+<pinref part="U1" gate="G$1" pin="XTAL_P/IO32"/>
 </segment>
 </net>
@@
 </segment>
 <segment>
-<pinref part="U1" gate="G$1" pin="IO35"/>
-<wire x1="63.5" y1="190.5" x2="60.96" y2="190.5" width="0.1524" layer="91"/>
-<label x="63.5" y="190.5" size="1.27" layer="95" xref="yes"/>
-</segment>
-</net>
+<wire x1="63.5" y1="195.58" x2="60.96" y2="195.58" width="0.1524" layer="91"/>
+<label x="63.5" y="195.58" size="1.27" layer="95" xref="yes"/>
+<pinref part="U1" gate="G$1" pin="XTAL_N/IO33"/>
+</segment>
+</net>
